File: projects/cali/cali.sch (EAGLE design)
At the start: 25 parts, among them Q3 IRF540, T1 BC547, T2 BC547, T3 BC547

Commit message: Board v1.0
Parts:
- removed Q3: IRF540, transistor-power:IRF540
- removed R15, R17: 10k, rcl:R-EU_0207/10
- removed R16: 1k, rcl:R-EU_0207/10
- removed R18: 10, rcl:R-EU_0207/10
- added D1: BAS316, nxp_60:BAS316
- added R11: 10k, rcl:R-EU_R1206
- added T4: IRLML2502, we-transistor:MOSFET-N-SOT23
- added U$4: FINDER-36.11, relay2:FINDER-36.11
- added X2: (no value), con-ptr500:AK500/4
- R1: value 0 -> 100; device rcl:R-EU_0207/10 -> rcl:R-EU_R1206
- R10: value 10k -> 1k; device rcl:R-EU_0207/10 -> rcl:R-EU_R1206
- R12: value 4k7 -> 1k; device rcl:R-EU_0207/10 -> rcl:R-EU_R1206
- R13: value 1k -> 0; device rcl:R-EU_0207/10 -> rcl:R-EU_R1206
- R14: value 10k -> 2k; device rcl:R-EU_0207/10 -> rcl:R-EU_R1206
- R2, R6: value 1k -> 100; device rcl:R-EU_0207/10 -> rcl:R-EU_R1206
- R3, R4, R5, R7, R8: device rcl:R-EU_0207/10 -> rcl:R-EU_R1206
- R9: value 1k -> 10k; device rcl:R-EU_0207/10 -> rcl:R-EU_R1206
- T1, T2: value BC547 -> IRLML2502; device transistor:BC547 -> we-transistor:MOSFET-N-SOT23
- T3: value BC547 -> 2N7002E; device transistor:BC547 -> nxp_60:2N7002E
Connections:
- removed net 5V0@1: U$2.5V0@1
- removed net N$16: Q3.G, R18.2
- removed net N$17: Q3.D, X1-11.KL
- removed net N$18: R12.1, U$2.GPIO26, X1-7.KL
- removed net N$20: U$2.GPIO21, X1-5.KL
- removed net N$21: U$2.GPIO20, X1-6.KL
- removed net N$22: R9.2, T3.B
- removed net N$23: R10.1, T3.C, X1-8.KL
- new net ADC0: U$1.A0
- new net ADC1: R7.1, R8.1, U$1.A1
- new net ADC2: R10.1, R9.1, U$1.A2
- new net ADC3: R11.1, R12.1, U$1.A3
- new net ADC4: R13.1, R14.1
- new net GPIO12: R6.1, U$2.GPIO12
- new net GPIO16: R1.1, U$2.GPIO16
- new net GPIO20: T2.S, U$2.GPIO20
- new net GPIO21: R5.1, T3.D, U$2.GPIO21
- new net GPIO26: U$2.GPIO26, X1-5.KL
- net +12V: now also D1.K, R3.2, R4.2, U$4G$1.+, X2-4.KL; no longer R10.2, R17.2, X1-10.KL
- net +3V3: now also R2.2, R5.2, X2-3.KL; no longer R12.2, R15.2, X1-9.KL
- net GND: now also R10.2, R12.2, R14.2, R8.2, T1.S, T4.S, U$2.GND@8, X2-1.KL, X2-2.KL; no longer Q3.S, R13.1, R4.1, R6.1, R8.1, T1.E, T2.E, T3.E
- net GPIO19: no longer R9.1
- net N$1: now also D1.A, T4.D, U$4G$1.-; no longer R1.1, X1-1.KL
- net N$10: now also R2.1, T2.G; no longer R14.1, T1.B
- net N$11: now also R3.1, T2.D, X1-10.KL; no longer R14.2, X1-12.KL
- net N$12: now also R4.1, T3.G; no longer R15.1, T1.C, U$2.GPIO16
- net N$13: now also T3.S, X1-9.KL; no longer R16.2, T2.B
- net N$14: now also R11.2, X1-3.KL; no longer R16.1, U$2.GPIO12
- net N$15: now also R13.2, X1-4.KL; no longer R17.1, R18.1, T2.C
- net N$2: now also T1.D, X1-11.KL; no longer R3.1, X1-2.KL
- net N$3: now also U$4G$2.S, X1-8.KL; no longer R5.1, X1-3.KL
- net N$4: now also R6.2, T4.G; no longer R7.1, X1-4.KL
- net N$5: now also U$4G$2.P, X1-6.KL; no longer R1.2, R2.2, U$1.A3
- net N$6: now also R1.2, T1.G; no longer R3.2, R4.2, U$1.A2
- net N$7: now also U$4G$2.O, X1-7.KL; no longer R13.2, R2.1
- net N$8: now also X1-1.KL; no longer R8.2, U$1.A0
- net N$9: now also R9.2, X1-2.KL; no longer R5.2, R6.2, U$1.A1
Other:
- note added: "ADC"
- note added: "Cali Board v1.0"
- note added: "Ladesignal"
- note added: "Lüfter"
- note added: "Raspi and Modules"
- note added: "Versorgung"
- note added: "Wechselrichter"

Commit message: Caliboard 1.0 routing done
Parts:
- added R15: 0, rcl:R-EU_R1206
- added X3, X4: (no value), con-ptr500:AK500/4
- X1: device con-ptr500:AK500/12 -> con-ptr500:AK500/4
Connections:
- removed net ADC4: R13.1, R14.1
- removed net N$14: R11.2, X1-3.KL
- removed net N$15: R13.2, X1-4.KL
- new net I_SOL: R13.2, X3-4.KL
- new net V_SOL: R7.2, X3-1.KL
- new net V_START: R11.2, X3-3.KL
- net ADC0: now also R7.1, R8.1
- net ADC1: now also R10.1, R9.1; no longer R7.1, R8.1
- net ADC2: now also R11.1, R12.1; no longer R10.1, R9.1
- net ADC3: now also R13.1, R14.1; no longer R11.1, R12.1
- net GPIO19: now also T2.S
- net GPIO20: no longer T2.S
- net GPIO26: now also X4-4.KL; no longer X1-5.KL
- net N$11: now also X1-3.KL; no longer X1-10.KL
- net N$13: now also R15.1, R9.2; no longer T3.S, X1-9.KL
- net N$2: now also X1-4.KL; no longer X1-11.KL
- net N$3: now also X4-3.KL; no longer X1-8.KL
- net N$5: now also X4-2.KL; no longer X1-6.KL
- net N$7: now also X4-1.KL; no longer X1-7.KL
- net N$8: now also T3.S, X1-2.KL; no longer R7.2, X1-1.KL
- net N$9: now also R15.2, X3-2.KL; no longer R9.2, X1-2.KL
Other:
- moved on the sheet: R9, X1-2, X1-3, X1-4

Commit message: Caliboard v1.1
- Change GPIOs to use GPIO of first row only
- Modify level shifter to sustain 12V
- Change GPIO for PWM
Connections:
- removed net N$12: R4.1, T3.G
- removed net N$8: T3.S, X1-2.KL
- new net CHGI: R5.1, T3.D, X1-2.KL
- new net GPIO10: T2.S, U$2.GPIO10/MOSI
- new net GPIO13: R1.1, U$2.GPIO13
- new net GPIO4: R6.1, U$2.GPIO4/GCKL
- new net GPIO9: U$2.GPIO9/MISO, X4-4.KL
- net +12V: now also R5.2; no longer R4.2
- net +3V3: now also R4.1, T3.G; no longer R5.2
- net GND: now also U$2.GND@1, U$2.GND@2, U$2.GND@4, U$2.GND@5, U$2.GND@6, U$2.GND@7
- net GPIO12: no longer R6.1
- net GPIO16: no longer R1.1
- net GPIO19: no longer T2.S
- net GPIO21: no longer R5.1, T3.D
- net GPIO26: now also R4.2, T3.S; no longer X4-4.KL
Other:
- note added: "Cali Board v1.1"
- note removed: "Cali Board v1.0"
- moved on the sheet: R4, X1-2
